Commit message: Add dog robot model and control interfaces

File: dog_bringup/xacro/dog.xacro (robot description, xacro)
@@ -46,8 +46,8 @@
         <origin xyz="0 0 0" rpy="0 0 0"/>
     </joint>
-    <xacro:dog_leg name="FL" mirror="1" f_b="1"/>
-    <xacro:dog_leg name="FR" mirror="-1" f_b="1"/>
-    <xacro:dog_leg name="HL" mirror="1" f_b="-1"/>
-    <xacro:dog_leg name="HR" mirror="-1" f_b="-1"/>
+    <xacro:dog_leg name="LF" mirror="1" f_b="1"/>
+    <xacro:dog_leg name="LH" mirror="1" f_b="-1"/>
+    <xacro:dog_leg name="RF" mirror="-1" f_b="1"/>
+    <xacro:dog_leg name="RH" mirror="-1" f_b="-1"/>
     <ros2_control name="dog_System" type="system">
         <hardware>
@@ -74,12 +74,12 @@
             <state_interface name="linear_acceleration_covariance"/>
         </sensor>
-        <sensor name="FL_contact_sensor"> <state_interface name="contact"/></sensor>
-        <sensor name="FR_contact_sensor"> <state_interface name="contact"/></sensor>
-        <sensor name="HL_contact_sensor"> <state_interface name="contact"/></sensor>
-        <sensor name="HR_contact_sensor"> <state_interface name="contact"/></sensor>
-        <xacro:leg_control_interface name="FL"/>
-        <xacro:leg_control_interface name="FR"/>
-        <xacro:leg_control_interface name="HL"/>
-        <xacro:leg_control_interface name="HR"/>
+        <sensor name="LF_contact_sensor"> <state_interface name="contact"/></sensor>
+        <sensor name="LH_contact_sensor"> <state_interface name="contact"/></sensor>
+        <sensor name="RF_contact_sensor"> <state_interface name="contact"/></sensor>
+        <sensor name="RH_contact_sensor"> <state_interface name="contact"/></sensor>
+        <xacro:leg_control_interface name="LF"/>
+        <xacro:leg_control_interface name="LH"/>
+        <xacro:leg_control_interface name="RF"/>
+        <xacro:leg_control_interface name="RH"/>
     </ros2_control>
     <gazebo reference="imu_link">
@@ -113,3 +113,16 @@
         </plugin>
     </gazebo>
+    <gazebo>
+      <plugin name="dog_ground_truth" filename="libgazebo_ros_p3d.so">
+        <ros>
+          <remapping>odom:=/ground_truth</remapping>
+        </ros>
+        <body_name>base_link</body_name>
+        <frame_name>world</frame_name>
+        <update_rate>1000.0</update_rate>
+        <xyz_offset>0 0 0</xyz_offset>
+        <rpy_offset>0 0 0</rpy_offset>
+        <gaussian_noise>0.001</gaussian_noise>
+      </plugin>
+    </gazebo>
 </robot>

File: dog_bringup/xacro/leg.xacro (robot description, xacro)
@@ -20,5 +20,5 @@
             </collision>
         </link>
-        <joint name="${name}_HipX_joint" type="revolute">
+        <joint name="${name}_HAA" type="revolute">
             <origin xyz="${f_b * hip_offset_x} ${mirror * hip_offset_y} 0"/>
             <parent link="TORSO"/>
@@ -46,5 +46,5 @@
             </collision>
         </link>
-        <joint name="${name}_HipY_joint" type="revolute">
+        <joint name="${name}_HFE" type="revolute">
             <origin xyz="0 ${mirror * thigh_offset_y} 0"/>
             <parent link="${name}_HIP"/>
@@ -78,5 +78,5 @@
             </collision>
         </link>
-        <joint name="${name}_Knee_joint" type="revolute">
+        <joint name="${name}_KFE" type="revolute">
             <origin xyz="0 0 ${shank_offset_z}"/>
             <parent link="${name}_THIGH"/>

File: dog_bringup/xacro/ros2_control.xacro (robot description, xacro)
@@ -2,5 +2,5 @@
 <robot xmlns:xacro="http://www.ros.org/wiki/xacro">
     <xacro:macro name="leg_control_interface" params="name">
-        <joint name="${name}_HipX_joint">
+        <joint name="${name}_HAA">
             <command_interface name="effort">
                 <param name="min">-${hipx_eff}</param>
@@ -19,5 +19,5 @@
             <state_interface name="effort"/>
         </joint>
-        <joint name="${name}_HipY_joint">
+        <joint name="${name}_HFE">
             <command_interface name="effort">
                 <param name="min">-${hipy_eff}</param>
@@ -36,5 +36,5 @@
             <state_interface name="effort"/>
         </joint>
-        <joint name="${name}_Knee_joint">
+        <joint name="${name}_KFE">
             <command_interface name="effort">
                 <param name="min">-${knee_eff}</param>

Commit message: 添加狗的世界配置文件，优化参数

File: dog_bringup/xacro/dog.xacro (robot description, xacro)
@@ -30,7 +30,7 @@
     <link name="imu_link">
         <inertial>
-            <mass value="0.001"/>
+            <mass value="0.1"/>
             <origin xyz="0 0 0" rpy="0 0 0"/>
-            <inertia ixx="1e-09" ixy="0.0" ixz="0.0" iyy="1e-09" iyz="0.0" izz="1e-09"/>
+            <inertia ixx="0.001" ixy="0.0" ixz="0.0" iyy="0.001" iyz="0.0" izz="0.001"/>
         </inertial>
     </link>
@@ -40,4 +40,7 @@
         <origin xyz="0 0 0" rpy="0 0 0"/>
     </joint>
+    <gazebo reference="imu_joint">
+            <preserveFixedJoint>true</preserveFixedJoint>
+    </gazebo>
     <link name="base_link"/>
     <joint name="base_joint" type="fixed">

File: dog_bringup/xacro/leg.xacro (robot description, xacro)
@@ -130,5 +130,7 @@
             <mu2>1.0</mu2>
             <kp>1000000.0</kp>
-            <kd>10000.0</kd>
+            <kd>1000.0</kd>
+            <minDepth>0.001</minDepth>
+            <maxVel>0.1</maxVel>
             <self_collide>1</self_collide>
             <sensor name="${name}_contact_sensor" type="contact">
